File: matenode.kicad_pcb (KiCad board)
At the start: 2 copper layers, 79 x 22 mm, 80 parts, among them J1 USB_C_Receptacle, J10 BAT_CONN, J2 VIN, J3 QWIIC, J4 VIN, J5 Lichtenprog_conn, J6 VIN, J7 VIN, J8 VIN, J9 SPK_OUT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

Commit message: finish routing. Now for aesthetics..
Parts:
- removed R11: 13k, Resistor_SMD:R_0402_1005Metric
- removed R4: 22k, Resistor_SMD:R_0402_1005Metric
- added C19: 10u, Capacitor_SMD:C_0402_1005Metric, F.Cu at (77.1, 74.8)
- J2, J6: moved to B.Cu
- R3: value 22k -> 10k
- U1: value SPX3819M5-L -> SPX3819M5-L-3-3
- U2: footprint Package_DFN_QFN:VQFN-16-1EP_3x3mm_P0.5mm_EP1.6x1.6mm -> Package_DFN_QFN:VQFN-16-1EP_3x3mm_P0.5mm_EP1.6x1.6mm_ThermalVias
- moved R26 21.3 mm to (70.4, 86.1), turned to 90 degrees
- moved R5 14.6 mm to (71.6, 86.3)
- moved R8 13.8 mm to (72.6, 86.3)
- moved C9 13.2 mm to (73.6, 86.3)
- moved C15 9.42 mm to (106.6, 79.3), turned to -90 degrees
- moved C18 7.58 mm to (109.2, 85.3), turned to -90 degrees
- moved R15 7.28 mm to (78.5, 72.4), turned to -90 degrees
- moved R24 7.18 mm to (77.4, 72.4), turned to 90 degrees
- moved C21 6.57 mm to (75.6, 88.3), turned to 90 degrees
- moved C16 6.16 mm to (78.5, 74.3)
- moved R20 5.21 mm to (76.7, 90.2), turned to -90 degrees
- moved R12 5.05 mm to (69.7, 76.3), turned to 0 degrees
- moved R25 4.79 mm to (76.4, 72.4), turned to -90 degrees
- moved R21 4.79 mm to (75.6, 90.2), turned to 90 degrees
- moved C12 4.20 mm to (90.7, 70.7)
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Connections:
- J10 pad 1: GND -> Net-(U2-Pad2)
- J10 pad 2: Net-(J10-Pad2) -> GND
- J9 pad 1: /SPK_OUTN -> /SPK_OUTP
- J9 pad 2: /SPK_OUTP -> /SPK_OUTN
- U1 pad 4: Net-(R11-Pad2) -> unconnected-(U1-Pad4)
- U2 pad 2: Net-(J10-Pad2) -> Net-(U2-Pad2)
- U2 pad 3: Net-(J10-Pad2) -> Net-(U2-Pad2)
Routing:
- net GND: track 30.7 -> 220.8 mm, vias 9 -> 30
- net +3.3V: track 33.2 -> 88.3 mm, vias 3 -> 5
- net /BOOT_BUT1: track 15.8 -> 52.6 mm, vias 2 -> 4
- net VBUS: track 8.80 -> 32.7 mm, vias 1 -> 5
- net /VBAT_MEAS: track 0.00 -> 20.5 mm, vias 0 -> 4
- net /PERIPH_ENA: track 37.9 -> 57.9 mm, vias 4 -> 3
- net +4V: track 0.00 -> 18.4 mm, vias 0 -> 11
- net /RTS: track 2.44 -> 18.8 mm, vias 0 -> 2
- net /IO_PERIPH_ENA: track 0.00 -> 12.6 mm, vias 0 -> 2
- net Net-(C13-Pad2): track 3.13 -> 13.0 mm, vias 0 -> 1
- net /DTR: track 4.70 -> 14.2 mm, vias 0 -> 2
- net Net-(D1-Pad1): track 0.00 -> 9.30 mm
- net Net-(Q4-Pad1): track 0.00 -> 8.09 mm
- net Net-(U2-Pad2): track 0.00 -> 7.72 mm
- net Net-(C21-Pad2): track 0.00 -> 7.15 mm
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- added copper zone on F.Cu, net +3.3V
- added copper zone on F.Cu, net GND
Other:
- board size 79 x 22 mm -> 76 x 22 mm
- board text added: "5V"
- board text added: "B1/BOOT"
- board text added: "B2/USER"
- board text added: "BATT+"
- board text added: "BATT-"
- board text added: "GND"
- board text added: "LiPo"
- board text added: "RST"
- board text added: "Spkr"

Commit message: finish silk, add prod files
Parts:
- added kibuzzard-6394BD6B: G***, kibuzzard-6394BD6B, B.Cu at (88.0, 77.3)
- added kibuzzard-6394BD6B: G***, kibuzzard-6394BD6B, B.Cu at (88.0, 74.8)
- added kibuzzard-6394BE40: G***, kibuzzard-6394BE40, B.Cu at (88.0, 89.8)
- added kibuzzard-6394BE58: G***, kibuzzard-6394BE58, B.Cu at (88.0, 84.9)
- added kibuzzard-6394BED6: G***, kibuzzard-6394BED6, B.Cu at (88.0, 87.4)
- added kibuzzard-6394BEEF: G***, kibuzzard-6394BEEF, B.Cu at (88.0, 79.8)
- added kibuzzard-6394BF0B: G***, kibuzzard-6394BF0B, B.Cu at (88.0, 82.4)
- added kibuzzard-6394BF19: G***, kibuzzard-6394BF19, B.Cu at (88.0, 72.3)
- added kibuzzard-6394C0D2: G***, kibuzzard-6394C0D2, B.Cu at (73.0, 72.5)
- added kibuzzard-6394C108: G***, kibuzzard-6394C108, B.Cu at (72.8, 89.1)
- added kibuzzard-6394C173: G***, kibuzzard-6394C173, B.Cu at (81.6, 80.8)
- added kibuzzard-6394C273: G***, kibuzzard-6394C273, B.Cu at (104.3, 73.8)
- added kibuzzard-6394C445: G***, kibuzzard-6394C445, B.Cu at (117.4, 73.1)
- added kibuzzard-6394C46A: G***, kibuzzard-6394C46A, B.Cu at (117.4, 75.1)
- added kibuzzard-6394C47E: G***, kibuzzard-6394C47E, B.Cu at (117.4, 77.0)
- added kibuzzard-6394C560: G***, kibuzzard-6394C560, B.Cu at (116.5, 71.2)
- added kibuzzard-6394C6B5: G***, kibuzzard-6394C6B5, F.Cu at (116.8, 80.1)
- added kibuzzard-6394C6E9: G***, kibuzzard-6394C6E9, F.Cu at (116.7, 81.8)
- added kibuzzard-6394C922: G***, kibuzzard-6394C922, B.Cu at (66.0, 78.4)
- added kibuzzard-6394C938: G***, kibuzzard-6394C938, B.Cu at (66.0, 83.8)
- added kibuzzard-6394CBE8: G***, kibuzzard-6394CBE8, F.Cu at (123.9, 72.7)
- added kibuzzard-6394CBE8: G***, kibuzzard-6394CBE8, B.Cu at (127.3, 72.7)
- added kibuzzard-6394CBFF: G***, kibuzzard-6394CBFF, F.Cu at (125.6, 78.6)
- added kibuzzard-6394CBFF: G***, kibuzzard-6394CBFF, B.Cu at (125.7, 78.6)
- added kibuzzard-6394CC15: G***, kibuzzard-6394CC15, F.Cu at (122.0, 84.6)
- added kibuzzard-6394CC15: G***, kibuzzard-6394CC15, B.Cu at (129.2, 84.6)
- added kibuzzard-6394D7BF: G***, kibuzzard-6394D7BF, B.Cu at (117.3, 86.3)
- moved JP4 0.55 mm to (81.5, 72.2)
- moved JP3 0.36 mm to (81.5, 89.8)
- moved D2 0.06 mm to (71.8, 72.2)
- turned D3 to -30 degrees
Routing:
- net GND: track 220.8 -> 228.3 mm
- net /PERIPH_ENA: track 57.9 -> 58.7 mm
Other:
- board text added: "OLED"
- board text added: "github.com/cr1tbit/matenode"
- board text removed: "B1/BOOT"
- board text removed: "B2/USER"
- board text removed: "LiPo"
- board text removed: "Spkr"

Commit message: final final
Parts:
- removed kibuzzard-6394CBFF (x2): G***, kibuzzard-6394CBFF
- added J11: 2.54 header, Connector_PinHeader_2.54mm:PinHeader_1x03_P2.54mm_Vertical, F.Cu at (128.0, 78.5)
- added kibuzzard-63966DAE: G***, kibuzzard-63966DAE, F.Cu at (122.2, 78.8)
- added kibuzzard-63966DAE: G***, kibuzzard-63966DAE, B.Cu at (122.3, 78.9)
- J4: value VIN -> Vout
- J7: value VIN -> Dout
- J8: value VIN -> Gout
- R12, R13, R14: footprint Resistor_SMD:R_0402_1005Metric -> Resistor_SMD:R_0603_1608Metric
- moved R1 9.43 mm to (74.0, 84.2), turned to -90 degrees
- moved kibuzzard-6394CC15 7.10 mm to (122.1, 84.8)
- moved R7 6.98 mm to (68.6, 75.9), turned to 180 degrees
- moved R13 6.88 mm to (77.4, 72.8), turned to -90 degrees
- moved R14 5.91 mm to (75.9, 72.8), turned to -90 degrees
- moved C17 4.11 mm to (78.6, 79.2), turned to -90 degrees
- moved C3 3.69 mm to (73.3, 78.1), turned to 0 degrees
- moved D1 3.56 mm to (71.8, 72.2)
- moved D2 3.50 mm to (68.8, 74.0)
- moved kibuzzard-6394CBE8 3.41 mm to (123.9, 73.0)
- moved R25 1.66 mm to (76.2, 70.8), turned to 180 degrees
- moved R24 1.60 mm to (78.7, 71.4)
- moved R6 1.10 mm to (74.2, 72.8)
- moved C19 1.00 mm to (76.1, 74.8)
- moved R15 0.96 mm to (78.7, 73.3)
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Routing:
- net Net-(R13-Pad2): track 1.17 -> 8.63 mm, vias 0 -> 2
- net Net-(D1-Pad1): track 9.37 -> 4.05 mm
- net +4V: track 18.4 -> 23.0 mm, vias 11 -> 12
- net Net-(D2-Pad1): track 6.04 -> 1.45 mm
- net /CC1: track 34.1 -> 30.7 mm
- net Net-(R14-Pad2): track 1.94 -> 5.13 mm, vias 0 -> 2
- net Net-(C19-Pad1): track 7.72 -> 5.10 mm
- net /IO_PERIPH_ENA: track 13.1 -> 11.4 mm
- net Net-(R7-Pad1): track 4.89 -> 3.30 mm, vias 2 -> 0
- net Net-(R6-Pad1): track 3.13 -> 1.70 mm
- net Net-(Q1-Pad1): track 7.53 -> 8.95 mm
- net unconnected-(U2-Pad14): track 1.31 -> 0.00 mm
- net VBUS: track 32.9 -> 31.9 mm
- net Net-(Q4-Pad1): track 8.09 -> 7.20 mm
- net /PERIPH_ENA: track 58.7 -> 59.5 mm
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