File: matenode.kicad_sch (KiCad schematic)
At the start: 80 parts, among them J1 USB_C_Receptacle, J10 BAT_CONN, J2 VIN, J3 QWIIC, J4 VIN, J5 Lichtenprog_conn, J6 VIN, J7 VIN, J8 VIN, J9 SPK_OUT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

Commit message: finish routing. Now for aesthetics..
Parts:
- removed R11: 13k, Resistor_SMD:R_0402_1005Metric, symbol Device:R_Small
- removed R4: 22k, Resistor_SMD:R_0402_1005Metric, symbol Device:R_Small
- removed U1: SPX3819M5-L, Package_TO_SOT_SMD:SOT-23-5, symbol Regulator_Linear:SPX3819M5-L
- added C19: 10u, Capacitor_SMD:C_0402_1005Metric, symbol Device:C_Small
- added U1: SPX3819M5-L-3-3, Package_TO_SOT_SMD:SOT-23-5, symbol Regulator_Linear:SPX3819M5-L-3-3
- R3: value 22k -> 10k
- U2: footprint Package_DFN_QFN:VQFN-16-1EP_3x3mm_P0.5mm_EP1.6x1.6mm -> Package_DFN_QFN:VQFN-16-1EP_3x3mm_P0.5mm_EP1.6x1.6mm_ThermalVias
Connections:
- net +3.3V: now also U1.5 (OUT)
- net +4V: now also U1.1 (IN)
- net GND: now also J10.2 (Pin_2), C19.2, U1.2 (GND); no longer J10.1 (Pin_1)
- net SPK_OUTN: now also J9.2 (Pin_2); no longer J9.1 (Pin_1)
- net SPK_OUTP: now also J9.1 (Pin_1); no longer J9.2 (Pin_2)
- net at U2.2 (BAT), U2.3 (BAT): now also J10.1 (Pin_1), C19.1; no longer J10.2 (Pin_2)
- net at R3.2: now also U1.3 (EN)
- no-connect marks 12 -> 13
Other:
- moved on the sheet: C22, D1, D2, R6, R7

Commit message: cleanup schematic
Other:
- note added: "Low / hiZ to disable periph power"
- note removed: "Low / hiZ to disable spkr and OLED"
- note removed: "VOUT = 1.235V x [1 + Ru/Rd] Rd must be >10k, Imax=500mA 3.3V: 22k/13k 1.8V: 22k/47k"

Commit message: final final
Parts:
- added J11: 2.54 header, Connector_PinHeader_2.54mm:PinHeader_1x03_P2.54mm_Vertical, symbol Connector_Generic:Conn_01x03
- J4: value VIN -> Vout
- J7: value VIN -> Dout
- J8: value VIN -> Gout
- R12, R13, R14: footprint Resistor_SMD:R_0402_1005Metric -> Resistor_SMD:R_0603_1608Metric
Connections:
- net +4V: now also J11.1 (Pin_1)
- net GND: now also J11.3 (Pin_3)
- net WS2812_OUT: now also J11.2 (Pin_2)
Other:
- moved on the sheet: J3, J4, J7, J8
